File: Tueroeffner.brd (EAGLE design)
At the start: 48.2 x 22.9 mm, 46 parts, among them IC1 IFX25001MEV33HTSA1, IC3 M25PE20, K2 EC2-12TNU, Q1 2N7002CK, Q2 2N7002CK

Commit message: Issue Text
Parts:
- moved JP2 0.48 mm to (0.00, 2.62)
Routing:
- net DC_5-12V: track 113.9 -> 114.9 mm
Other:
- board size 48.2 x 22.9 mm -> 48.7 x 22.9 mm
- board text added: "Check C7 Footprint! Check 330Ohm Footprint!"
Changed lines of the file:
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@@
 <layers>
 <layer number="1" name="Top" color="4" fill="1" visible="yes" active="yes"/>
-<layer number="16" name="Bottom" color="1" fill="1" visible="yes" active="yes"/>
+<layer number="16" name="Bottom" color="1" fill="1" visible="no" active="yes"/>
 <layer number="17" name="Pads" color="2" fill="1" visible="yes" active="yes"/>
 <layer number="18" name="Vias" color="2" fill="1" visible="yes" active="yes"/>
@@
 <layer number="20" name="Dimension" color="15" fill="1" visible="yes" active="yes"/>
 <layer number="21" name="tPlace" color="7" fill="1" visible="yes" active="yes"/>
-<layer number="22" name="bPlace" color="7" fill="1" visible="yes" active="yes"/>
+<layer number="22" name="bPlace" color="7" fill="1" visible="no" active="yes"/>
 <layer number="23" name="tOrigins" color="15" fill="1" visible="yes" active="yes"/>
-<layer number="24" name="bOrigins" color="15" fill="1" visible="yes" active="yes"/>
+<layer number="24" name="bOrigins" color="15" fill="1" visible="no" active="yes"/>
 <layer number="25" name="tNames" color="7" fill="1" visible="yes" active="yes"/>
-<layer number="26" name="bNames" color="7" fill="1" visible="yes" active="yes"/>
+<layer number="26" name="bNames" color="7" fill="1" visible="no" active="yes"/>
 <layer number="27" name="tValues" color="7" fill="1" visible="no" active="yes"/>
 <layer number="28" name="bValues" color="7" fill="1" visible="no" active="yes"/>
 <layer number="29" name="tStop" color="7" fill="3" visible="yes" active="yes"/>
-<layer number="30" name="bStop" color="7" fill="6" visible="yes" active="yes"/>
+<layer number="30" name="bStop" color="7" fill="6" visible="no" active="yes"/>
 <layer number="31" name="tCream" color="7" fill="4" visible="yes" active="yes"/>
-<layer number="32" name="bCream" color="7" fill="5" visible="yes" active="yes"/>
+<layer number="32" name="bCream" color="7" fill="5" visible="no" active="yes"/>
 <layer number="33" name="tFinish" color="6" fill="3" visible="no" active="yes"/>
 <layer number="34" name="bFinish" color="6" fill="6" visible="no" active="yes"/>
@@
 <layer number="38" name="bTest" color="7" fill="1" visible="no" active="yes"/>
 <layer number="39" name="tKeepout" color="4" fill="11" visible="yes" active="yes"/>
-<layer number="40" name="bKeepout" color="1" fill="11" visible="yes" active="yes"/>
+<layer number="40" name="bKeepout" color="1" fill="11" visible="no" active="yes"/>
 <layer number="41" name="tRestrict" color="4" fill="10" visible="yes" active="yes"/>
-<layer number="42" name="bRestrict" color="1" fill="10" visible="yes" active="yes"/>
+<layer number="42" name="bRestrict" color="1" fill="10" visible="no" active="yes"/>
 <layer number="43" name="vRestrict" color="2" fill="10" visible="no" active="yes"/>
 <layer number="44" name="Drills" color="7" fill="1" visible="no" active="yes"/>
@@
 <layer number="50" name="dxf" color="7" fill="1" visible="no" active="no"/>
 <layer number="51" name="tDocu" color="7" fill="1" visible="yes" active="yes"/>
-<layer number="52" name="bDocu" color="7" fill="1" visible="yes" active="yes"/>
+<layer number="52" name="bDocu" color="7" fill="1" visible="no" active="yes"/>
 <layer number="53" name="tGND_GNDA" color="7" fill="1" visible="no" active="no"/>
 <layer number="54" name="bGND_GNDA" color="7" fill="1" visible="no" active="no"/>
@@
 <board>
 <plain>
-<wire x1="-1.5875" y1="-1.27" x2="46.66" y2="-1.27" width="0" layer="20"/>
-<wire x1="46.66" y1="21.58" x2="-1.5875" y2="21.58" width="0" layer="20"/>
-<wire x1="-1.5875" y1="21.58" x2="-1.5875" y2="-1.27" width="0" layer="20"/>
+<wire x1="-2.06375" y1="-1.27" x2="46.66" y2="-1.27" width="0" layer="20"/>
+<wire x1="46.66" y1="21.58" x2="-2.06375" y2="21.58" width="0" layer="20"/>
+<wire x1="-2.06375" y1="21.58" x2="-2.06375" y2="-1.27" width="0" layer="20"/>
 <dimension x1="0" y1="0" x2="0" y2="20" x3="-2" y3="10" textsize="1.778" layer="47"/>
 <dimension x1="0" y1="0" x2="50" y2="0" x3="25" y3="-4" textsize="1.778" layer="47"/>
@@
 DoorOpener v1.1</text>
 <wire x1="46.66" y1="-1.27" x2="46.66" y2="21.59" width="0" layer="20"/>
+<text x="3.095625" y="23.495" size="1.778" layer="1">Check C7 Footprint!
+Check 330Ohm Footprint!</text>
 </plain>
 <attributes>
@@
 <attribute name="VALUE" x="18.201875" y="9.404375" size="1.27" layer="27" rot="R270"/>
 </element>
-<element name="JP2" library="SparkFun-Connectors" package="SCREWTERMINAL-3.5MM-4" value="" x="0.47625" y="2.619375" smashed="yes" rot="R90">
-<attribute name="NAME" x="2.69875" y="0.15875" size="0.8128" layer="25" rot="R90"/>
-<attribute name="VALUE" x="-0.79375" y="1.349375" size="0.4064" layer="27" rot="R90"/>
+<element name="JP2" library="SparkFun-Connectors" package="SCREWTERMINAL-3.5MM-4" value="" x="0" y="2.619375" smashed="yes" rot="R90">
+<attribute name="NAME" x="2.2225" y="0.15875" size="0.8128" layer="25" rot="R90"/>
+<attribute name="VALUE" x="-1.27" y="1.349375" size="0.4064" layer="27" rot="R90"/>
 </element>
 <element name="JP3" library="SparkFun-Connectors" package="SCREWTERMINAL-3.5MM-4" value="" x="44.053125" y="2.619375" smashed="yes" rot="R90">
@@
 <contactref element="C7" pad="-"/>
 <polygon width="0.4064" layer="16">
-<vertex x="-1.5875" y="-1.27"/>
+<vertex x="-2.06375" y="-1.27"/>
 <vertex x="46.99" y="-1.27"/>
 <vertex x="46.99" y="21.59"/>
-<vertex x="-1.5875" y="21.59"/>
+<vertex x="-2.06375" y="21.59"/>
 </polygon>
 <polygon width="0.4064" layer="1" rank="2">
-<vertex x="-1.5875" y="-1.27"/>
+<vertex x="-2.06375" y="-1.27"/>
 <vertex x="46.99" y="-1.27"/>
 <vertex x="46.99" y="21.59"/>
-<vertex x="-1.5875" y="21.59"/>
+<vertex x="-2.06375" y="21.59"/>
 </polygon>
 <contactref element="JP2" pad="3"/>
@@
 <via x="16.430625" y="18.25625" extent="1-16" drill="0.3"/>
 <via x="17.224375" y="14.684375" extent="1-16" drill="0.3"/>
+<via x="19.3675" y="4.92125" extent="1-16" drill="0.3"/>
+<polygon width="0.4064" layer="1" thermals="no" rank="2">
+<vertex x="13.255625" y="18.335625"/>
+<vertex x="15.954375" y="18.335625"/>
+<vertex x="15.954375" y="13.890625"/>
+<vertex x="13.255625" y="13.890625"/>
+</polygon>
 </signal>
 <signal name="DC_5-12V">
@@
 <contactref element="K2" pad="8"/>
 <via x="13.17625" y="2.54" extent="1-16" drill="0.6"/>
-<wire x1="0.47625" y1="17.619375" x2="0.47625" y2="15.795625" width="0.8128" layer="16"/>
-<wire x1="0.47625" y1="15.795625" x2="2.69875" y2="13.573125" width="0.8128" layer="16"/>
-<wire x1="2.69875" y1="13.573125" x2="2.69875" y2="1.905" width="0.8128" layer="16"/>
-<wire x1="3.33375" y1="1.27" x2="11.58875" y2="1.27" width="0.8128" layer="16"/>
+<wire x1="0" y1="17.619375" x2="0" y2="15.795625" width="0.8128" layer="16"/>
+<wire x1="0" y1="15.795625" x2="2.2225" y2="13.573125" width="0.8128" layer="16"/>
+<wire x1="2.2225" y1="13.573125" x2="2.2225" y2="1.905" width="0.8128" layer="16"/>
+<wire x1="2.8575" y1="1.27" x2="11.58875" y2="1.27" width="0.8128" layer="16"/>
 <wire x1="33.655" y1="12.22375" x2="38.735" y2="12.22375" width="0.8128" layer="16"/>
 <wire x1="38.735" y1="12.22375" x2="38.735" y2="14.76375" width="0.8128" layer="16"/>
 <wire x1="38.735" y1="12.22375" x2="39.52875" y2="12.22375" width="0.8128" layer="1"/>
 <wire x1="41.5925" y1="10.16" x2="41.5925" y2="5.08" width="0.8128" layer="1"/>
-<wire x1="3.33375" y1="1.27" x2="2.69875" y2="1.905" width="0.8128" layer="16"/>
+<wire x1="2.8575" y1="1.27" x2="2.2225" y2="1.905" width="0.8128" layer="16"/>
 <wire x1="44.053125" y1="2.619375" x2="39.290625" y2="2.619375" width="0.8128" layer="16"/>
 <wire x1="39.290625" y1="2.619375" x2="38.735" y2="2.06375" width="0.8128" layer="16"/>
@@
 <wire x1="41.5925" y1="10.16" x2="39.52875" y2="12.22375" width="0.8128" layer="1"/>
 <wire x1="8.264775" y1="18.37435" x2="3.889375" y2="18.37435" width="0.8128" layer="1"/>
-<wire x1="3.889375" y1="18.37435" x2="1.231225" y2="18.37435" width="0.8128" layer="1"/>
-<wire x1="1.231225" y1="18.37435" x2="0.47625" y2="17.619375" width="0.8128" layer="1"/>
+<wire x1="3.889375" y1="18.37435" x2="0.754975" y2="18.37435" width="0.8128" layer="1"/>
+<wire x1="0.754975" y1="18.37435" x2="0" y2="17.619375" width="0.8128" layer="1"/>
 <contactref element="R6" pad="1"/>
 <wire x1="3.96875" y1="11.509375" x2="3.96875" y2="18.294975" width="0.4064" layer="1"/>
@@
 <contactref element="R2" pad="2"/>
 <contactref element="JP2" pad="2"/>
-<wire x1="0.47625" y1="7.619375" x2="5.066875" y2="7.619375" width="0.8128" layer="1"/>
+<wire x1="0" y1="7.619375" x2="5.066875" y2="7.619375" width="0.8128" layer="1"/>
 <wire x1="5.066875" y1="7.619375" x2="5.239375" y2="7.55375" width="0.8128" layer="1"/>
 </signal>
@@
 <contactref element="JP2" pad="1"/>
 <contactref element="B1" pad="AC1"/>
-<wire x1="0.47625" y1="2.619375" x2="3.580625" y2="2.619375" width="0.8128" layer="1"/>
+<wire x1="0" y1="2.619375" x2="3.580625" y2="2.619375" width="0.8128" layer="1"/>
 <wire x1="3.580625" y1="2.619375" x2="4.924375" y2="1.275625" width="0.8128" layer="1"/>
 </signal>
